File: hardware/mixsid.sch (KiCad schematic (older format))
At the start: 69 parts, among them P1 INPUT, P2 CONTROL, P4 SOCKET LEFT, P5 OUTPUT, P6 SOCKET RIGHT, Q1 BC547, Q2 BC547, U1 GAL16V8, U2 SID2, U3 7812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

Commit message: Hardware: Improved routing, silkscreen
Parts:
- P2: footprint Pin_Headers:Pin_Header_Straight_2x07 -> Pinheaders:Pin_Header_Straight_2x07
Changed lines of the file:
@@
 F 0 "P2" H 1200 2450 50  0000 C CNN
 F 1 "CONTROL" V 1200 2050 50  0000 C CNN
-F 2 "Pin_Headers:Pin_Header_Straight_2x07" H 1200 850 60  0001 C CNN
+F 2 "Pinheaders:Pin_Header_Straight_2x07" H 1200 850 60  0001 C CNN
 F 3 "" H 1200 850 60  0000 C CNN
 	1    1200 2050

Commit message: Hardware: Use rect pots for digifix again, placed volume pods horizontally
Parts:
- P2: footprint Pinheaders:Pin_Header_Straight_2x07 -> Pin_Headers:Pin_Header_Straight_2x07
- RV1, RV2: footprint Potentiometers:Potentiometer_Bourns_3339P_Angular_ScrewUp -> Potentiometers:Potentiometer_Bourns_3296W_3-8Zoll_Inline_ScrewUp
Changed lines of the file:
@@
 F 0 "RV1" H 5100 5650 50  0000 C CNN
 F 1 "1M" H 5100 5750 50  0000 C CNN
-F 2 "Potentiometers:Potentiometer_Bourns_3339P_Angular_ScrewUp" H 5100 5750 60  0001 C CNN
+F 2 "Potentiometers:Potentiometer_Bourns_3296W_3-8Zoll_Inline_ScrewUp" H 5100 5750 60  0001 C CNN
 F 3 "" H 5100 5750 60  0000 C CNN
 	1    5100 5750
@@
 F 0 "RV2" H 2150 5650 50  0000 C CNN
 F 1 "1M" H 2150 5750 50  0000 C CNN
-F 2 "Potentiometers:Potentiometer_Bourns_3339P_Angular_ScrewUp" H 2150 5750 60  0001 C CNN
+F 2 "Potentiometers:Potentiometer_Bourns_3296W_3-8Zoll_Inline_ScrewUp" H 2150 5750 60  0001 C CNN
 F 3 "" H 2150 5750 60  0000 C CNN
 	1    2150 5750
@@
 F 0 "P2" H 1200 2450 50  0000 C CNN
 F 1 "CONTROL" V 1200 2050 50  0000 C CNN
-F 2 "Pinheaders:Pin_Header_Straight_2x07" H 1200 850 60  0001 C CNN
+F 2 "Pin_Headers:Pin_Header_Straight_2x07" H 1200 850 60  0001 C CNN
 F 3 "" H 1200 850 60  0000 C CNN
 	1    1200 2050

Commit message: Hardware: Use round pots fot digifix as well
Parts:
- RV1, RV2: footprint Potentiometers:Potentiometer_Bourns_3296W_3-8Zoll_Inline_ScrewUp -> Potentiometers:Potentiometer_Bourns_3339P_Angular_ScrewUp
Changed lines of the file:
@@
 F 0 "RV1" H 5100 5650 50  0000 C CNN
 F 1 "1M" H 5100 5750 50  0000 C CNN
-F 2 "Potentiometers:Potentiometer_Bourns_3296W_3-8Zoll_Inline_ScrewUp" H 5100 5750 60  0001 C CNN
+F 2 "Potentiometers:Potentiometer_Bourns_3339P_Angular_ScrewUp" H 5100 5750 60  0001 C CNN
 F 3 "" H 5100 5750 60  0000 C CNN
 	1    5100 5750
@@
 F 0 "RV2" H 2150 5650 50  0000 C CNN
 F 1 "1M" H 2150 5750 50  0000 C CNN
-F 2 "Potentiometers:Potentiometer_Bourns_3296W_3-8Zoll_Inline_ScrewUp" H 2150 5750 60  0001 C CNN
+F 2 "Potentiometers:Potentiometer_Bourns_3339P_Angular_ScrewUp" H 2150 5750 60  0001 C CNN
 F 3 "" H 2150 5750 60  0000 C CNN
 	1    2150 5750
